Commit message: feature/update-urdf-and-add-bringup

File: kimm_wheel_legged_robot_description/urdf/kimm_wheel_legged_robot_drive.urdf (robot description, URDF)
Before this commit: robot kimm_wheel_legged_robot, 27 links, 26 joints
Links:
- removed link base_aligned
- added link pelvis, mass 0.8; collision mesh filename=file://$(find kimm_wheel_legged_robot_description)/meshes/p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 scale=0.001 0.001 0.001; visual mesh filename=file://$(find kimm_wheel_legged_robot_description)/meshes/p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 scale=0.001 0.001 0.001
- link base_link: mass 1.0607603720590608 -> None; geometry 
- link left_ankle_link: mass 0.6291183093975233 -> 0.3; geometry collision mesh filename=file://$(find kimm_wheel_legged_robot_description)/meshes/l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 scale=0.001 0.001 0.001; visual mesh filename=file://$(find kimm_wheel_legged_robot_description)/meshes/l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 scale=0.001 0.001 0.001
- link left_foot_link: mass 1.1702691153174818 -> 0.6; geometry collision mesh filename=file://$(find kimm_wheel_legged_robot_description)/meshes/l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 scale=0.001 0.001 0.001; visual mesh filename=file://$(find kimm_wheel_legged_robot_description)/meshes/l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 scale=0.001 0.001 0.001
- link left_foot_wheel_L: mass 0.030061819599063008 -> 0.15; geometry collision mesh filename=file://$(find kimm_wheel_legged_robot_description)/meshes/l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 scale=0.001 0.001 0.001; visual mesh filename=file://$(find kimm_wheel_legged_robot_description)/meshes/l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 scale=0.001 0.001 0.001
- link left_foot_wheel_R: mass 0.030061819599062962 -> 0.15; geometry collision mesh filename=file://$(find kimm_wheel_legged_robot_description)/meshes/l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 scale=0.001 0.001 0.001; visual mesh filename=file://$(find kimm_wheel_legged_robot_description)/meshes/l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 scale=0.001 0.001 0.001
- link left_hip_pitch_link: mass 4.43199564289481 -> 1.0; geometry collision mesh filename=file://$(find kimm_wheel_legged_robot_description)/meshes/l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 scale=0.001 0.001 0.001; visual mesh filename=file://$(find kimm_wheel_legged_robot_description)/meshes/l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 scale=0.001 0.001 0.001
- link left_hip_roll_link: mass 4.081497564698486 -> 1.0; geometry collision mesh filename=file://$(find kimm_wheel_legged_robot_description)/meshes/l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 scale=0.001 0.001 0.001; visual mesh filename=file://$(find kimm_wheel_legged_robot_description)/meshes/l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 scale=0.001 0.001 0.001
- link left_hip_yaw_link: mass 4.470572358545368 -> 1.0; geometry collision mesh filename=file://$(find kimm_wheel_legged_robot_description)/meshes/l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 scale=0.001 0.001 0.001; visual mesh filename=file://$(find kimm_wheel_legged_robot_description)/meshes/l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 scale=0.001 0.001 0.001
- link left_knee_link: mass 6.932201355092377 -> 3.0; geometry collision mesh filename=file://$(find kimm_wheel_legged_robot_description)/meshes/l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 scale=0.001 0.001 0.001; visual mesh filename=file://$(find kimm_wheel_legged_robot_description)/meshes/l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 scale=0.001 0.001 0.001
- link left_long_tendon_connector_link: geometry collision mesh filename=file://$(find kimm_wheel_legged_robot_description)/meshes/l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 scale=0.001 0.001 0.001; visual mesh filename=file://$(find kimm_wheel_legged_robot_description)/meshes/l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 scale=0.001 0.001 0.001
- link left_short_tendon_connector_link: geometry collision mesh filename=file://$(find kimm_wheel_legged_robot_description)/meshes/l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 scale=0.001 0.001 0.001; visual mesh filename=file://$(find kimm_wheel_legged_robot_description)/meshes/l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 scale=0.001 0.001 0.001
- link left_thigh_wheel_link: mass 11.776367101859407 -> 2.0; geometry collision mesh filename=file://$(find kimm_wheel_legged_robot_description)/meshes/l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 scale=0.001 0.001 0.001; visual mesh filename=file://$(find kimm_wheel_legged_robot_description)/meshes/l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 scale=0.001 0.001 0.001
- link left_wheel: mass 6.388977469824551 -> 1.2; geometry collision mesh filename=file://$(find kimm_wheel_legged_robot_description)/meshes/l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 scale=0.001 0.001 0.001; visual mesh filename=file://$(find kimm_wheel_legged_robot_description)/meshes/l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 scale=0.001 0.001 0.001
- link right_ankle_link: mass 0.6291183093975233 -> 0.3; geometry collision mesh filename=file://$(find kimm_wheel_legged_robot_description)/meshes/r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 scale=0.001 0.001 0.001; visual mesh filename=file://$(find kimm_wheel_legged_robot_description)/meshes/r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 scale=0.001 0.001 0.001
- link right_foot_link: mass 1.1702691153174818 -> 0.6; geometry collision mesh filename=file://$(find kimm_wheel_legged_robot_description)/meshes/r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 scale=0.001 0.001 0.001; visual mesh filename=file://$(find kimm_wheel_legged_robot_description)/meshes/r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 scale=0.001 0.001 0.001
- link right_foot_wheel_L: mass 0.030061819599062962 -> 0.15; geometry collision mesh filename=file://$(find kimm_wheel_legged_robot_description)/meshes/r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 scale=0.001 0.001 0.001; visual mesh filename=file://$(find kimm_wheel_legged_robot_description)/meshes/r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 scale=0.001 0.001 0.001
- link right_foot_wheel_R: mass 0.030061819599063008 -> 0.15; geometry collision mesh filename=file://$(find kimm_wheel_legged_robot_description)/meshes/r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 scale=0.001 0.001 0.001; visual mesh filename=file://$(find kimm_wheel_legged_robot_description)/meshes/r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 scale=0.001 0.001 0.001
- link right_hip_pitch_link: mass 4.43199564289481 -> 1.0; geometry collision mesh filename=file://$(find kimm_wheel_legged_robot_description)/meshes/r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 scale=0.001 0.001 0.001; visual mesh filename=file://$(find kimm_wheel_legged_robot_description)/meshes/r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 scale=0.001 0.001 0.001
- link right_hip_roll_link: mass 4.081497564698486 -> 1.0; geometry collision mesh filename=file://$(find kimm_wheel_legged_robot_description)/meshes/r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 scale=0.001 0.001 0.001; visual mesh filename=file://$(find kimm_wheel_legged_robot_description)/meshes/r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 scale=0.001 0.001 0.001
- link right_hip_yaw_link: mass 4.4705723411131935 -> 1.0; geometry collision mesh filename=file://$(find kimm_wheel_legged_robot_description)/meshes/r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 scale=0.001 0.001 0.001; visual mesh filename=file://$(find kimm_wheel_legged_robot_description)/meshes/r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 scale=0.001 0.001 0.001
- link right_knee_link: mass 6.932201355092377 -> 3.0; geometry collision mesh filename=file://$(find kimm_wheel_legged_robot_description)/meshes/r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 scale=0.001 0.001 0.001; visual mesh filename=file://$(find kimm_wheel_legged_robot_description)/meshes/r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 scale=0.001 0.001 0.001
- link right_long_tendon_connector_link: geometry collision mesh filename=file://$(find kimm_wheel_legged_robot_description)/meshes/r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 scale=0.001 0.001 0.001; visual mesh filename=file://$(find kimm_wheel_legged_robot_description)/meshes/r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 scale=0.001 0.001 0.001
- link right_short_tendon_connector_link: geometry collision mesh filename=file://$(find kimm_wheel_legged_robot_description)/meshes/r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 scale=0.001 0.001 0.001; visual mesh filename=file://$(find kimm_wheel_legged_robot_description)/meshes/r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 scale=0.001 0.001 0.001
- link right_thigh_wheel_link: mass 11.776367101859407 -> 2.0; geometry collision mesh filename=file://$(find kimm_wheel_legged_robot_description)/meshes/r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 scale=0.001 0.001 0.001; visual mesh filename=file://$(find kimm_wheel_legged_robot_description)/meshes/r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 scale=0.001 0.001 0.001
- link right_wheel: mass 6.388977469824551 -> 1.2; geometry collision mesh filename=file://$(find kimm_wheel_legged_robot_description)/meshes/r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 scale=0.001 0.001 0.001; visual mesh filename=file://$(find kimm_wheel_legged_robot_description)/meshes/r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 scale=0.001 0.001 0.001
- link torso_link: mass 57.103267228355826 -> 15.0; geometry collision mesh filename=file://$(find kimm_wheel_legged_robot_description)/meshes/t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 scale=0.001 0.001 0.001; visual mesh filename=file://$(find kimm_wheel_legged_robot_description)/meshes/t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 scale=0.001 0.001 0.001
Joints:
- removed joint base_link_to_base_aligned
- added joint base_link_to_pelvis: type fixed, parent base_link, child pelvis, origin xyz=0 0 0 rpy=1.5708 0 -1.5708
- joint left_pelvis_joint: parent base_link -> pelvis
- joint right_pelvis_joint: parent base_link -> pelvis
- joint torso_joint: parent base_link -> pelvis

File: kimm_wheel_legged_robot_description/urdf/kimm_wheel_legged_robot_walk.urdf (robot description, URDF)
Before this commit: robot kimm_wheel_legged_robot, 27 links, 26 joints
Links:
- removed link base_aligned
- added link pelvis, mass 0.8; collision mesh filename=package://kimm_wheel_legged_robot_description/meshes/pelvis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 scale=0.001 0.001 0.001; visual mesh filename=package://kimm_wheel_legged_robot_description/meshes/pelvis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 scale=0.001 0.001 0.001
- link base_link: mass 1.0607603720590608 -> None; geometry 
- link left_ankle_link: mass 0.6291183093975233 -> 0.3
- link left_foot_link: mass 1.1702691153174818 -> 0.6
- link left_foot_wheel_L: mass 0.030061819599063008 -> 0.15
- link left_foot_wheel_R: mass 0.030061819599062962 -> 0.15
- link left_hip_pitch_link: mass 4.43199564289481 -> 1.0
- link left_hip_roll_link: mass 4.081497564698486 -> 1.0
- link left_hip_yaw_link: mass 4.470572358545368 -> 1.0
- link left_knee_link: mass 6.932201355092377 -> 3.0
- link left_thigh_wheel_link: mass 11.776367101859407 -> 2.0
- link left_wheel: mass 6.388977469824551 -> 1.2
- link right_ankle_link: mass 0.6291183093975233 -> 0.3
- link right_foot_link: mass 1.1702691153174818 -> 0.6
- link right_foot_wheel_L: mass 0.030061819599062962 -> 0.15
- link right_foot_wheel_R: mass 0.030061819599063008 -> 0.15
- link right_hip_pitch_link: mass 4.43199564289481 -> 1.0
- link right_hip_roll_link: mass 4.081497564698486 -> 1.0
- link right_hip_yaw_link: mass 4.4705723411131935 -> 1.0
- link right_knee_link: mass 6.932201355092377 -> 3.0
- link right_thigh_wheel_link: mass 11.776367101859407 -> 2.0
- link right_wheel: mass 6.388977469824551 -> 1.2
- link torso_link: mass 57.103267228355826 -> 15.0
Joints:
- removed joint base_link_to_base_aligned
- added joint base_link_to_pelvis: type fixed, parent base_link, child pelvis, origin xyz=0 0 0 rpy=1.5708 0 -1.5708
- joint left_pelvis_joint: parent base_link -> pelvis
- joint right_pelvis_joint: parent base_link -> pelvis
- joint torso_joint: parent base_link -> pelvis
